File: hardware/sounddecoder-esp32-s3-wroom-2/sounddecoder-esp32-s3-wroom-2.kicad_pcb (KiCad board)
At the start: 4 copper layers, 42.5 x 59.8 mm, 34 parts, among them J1 Input power, J10 AUX1, J11 AUX2, J12 AUX3, J13 AUX4, J3 Motor, J4 Speaker, J5 DEBUG, J6 Conn_01x03_Pin, J7 Smoke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

Commit message: Many changes
Parts:
- moved J13 4.28 mm to (110.8, 117.0)
- moved J12 3.54 mm to (110.8, 111.0)
- moved J11 2.75 mm to (110.8, 105.0)
- moved J10 2.03 mm to (110.8, 99.0)
- moved J9 1.29 mm to (110.8, 93.0)
- moved J8 0.54 mm to (110.8, 87.0)
- moved J7 0.21 mm to (110.8, 81.0)
Routing:
- net Net-(J13-Pin_2): track 27.0 -> 22.7 mm
- net Net-(J12-Pin_2): track 20.8 -> 18.1 mm
- net +5V: track 61.1 -> 62.2 mm
- net Net-(J11-Pin_2): track 15.6 -> 16.7 mm
- net Net-(J10-Pin_2): track 15.9 -> 16.7 mm
- net /BackLED: track 19.4 -> 19.9 mm
