File: hardware/sounddecoder-esp32-s3-wroom-2-micro/sounddecoder-esp32-s3-wroom-2-micro.kicad_sch (KiCad schematic)
At the start: 48 parts, among them J1 Pins, J2 Conn_01x02_Pin, J3 TrackRight, J4 Smoke_Pin, J5 TrackLeft, U1 TPS54302, U2 DRV8235, U3 MAX98357A, U7 ESP32-S3-WROOM-2, U8 ULN2003A

Commit message: Many updates
Other:
- moved on the sheet: D1, D2, D3, D4, J3, J5, R4, R5
