File: hardware/sounddecoder-esp32-s3-wroom-2-micro/sounddecoder-esp32-s3-wroom-2-micro.kicad_pcb (KiCad board)
At the start: 4 copper layers, 22.5 x 49.5 mm, 39 parts, among them J1 Pins, J2 Conn_01x02_Pin, J4 Smoke_Pin, U1 TPS563202S, U3 MAX98357A, U4 DRV8251A, U7 ESP32-S3-WROOM-2, U8 ULN2003A

Commit message: Updated micro decode board
Parts:
- removed C21: 10uF, Capacitor_SMD:C_0603_1608Metric
- removed U4: DRV8251A, Package_SO:Texas_HSOP-8-1EP_3.9x4.9mm_P1.27mm_ThermalVias
- added C6: 0.1uF, Capacitor_SMD:C_0603_1608Metric, F.Cu at (98.5, 117.5)
- added D1: PMEG2020EJ, Diode_SMD:D_SOD-323, F.Cu at (104.0, 112.3)
- added D2: PMEG2020EJ, Diode_SMD:D_SOD-323, F.Cu at (104.0, 108.5)
- added D3: PMEG2020EJ, Diode_SMD:D_SOD-323, F.Cu at (104.0, 110.4)
- added D4: PMEG2020EJ, Diode_SMD:D_SOD-323, F.Cu at (104.0, 114.2)
- added J3: TrackRight, TestPoint:TestPoint_THTPad_1.0x1.0mm_Drill0.5mm, F.Cu at (104.6, 106.5)
- added J5: TrackLeft, TestPoint:TestPoint_THTPad_1.0x1.0mm_Drill0.5mm, F.Cu at (104.6, 116.2)
- added R17: 1k, Capacitor_SMD:C_0603_1608Metric, F.Cu at (91.6, 116.7)
- added R18: 2.2k, Capacitor_SMD:C_0603_1608Metric, F.Cu at (104.3, 99.8)
- added R19: 2.2k, Capacitor_SMD:C_0603_1608Metric, F.Cu at (104.3, 98.4)
- added U2: DRV8235, Package_DFN_QFN:WQFN-16-1EP_3x3mm_P0.5mm_EP1.68x1.68mm_ThermalVias, F.Cu at (95.5, 116.9)
- C3: value 33pF -> 47pF
- L1: value 3.3uH -> 6.8uH
- R1: value 1k -> 10k
- R10: value 10k -> 22.1k
- R4: value 15k -> 75kΩ
- R5: value 15k -> 20kΩ
- R6: value 1k -> 105k
- R7: value 1k -> 49.9
- R8: value 10k -> 511k
- R9: value 31k -> 100k
- U1: value TPS563202S -> TPS54302; footprint Package_TO_SOT_SMD:SOT-563 -> Package_TO_SOT_SMD:SOT-23-6
- moved R5 19.2 mm to (101.1, 104.7), turned to 180 degrees
- moved R6 18.8 mm to (92.2, 112.5), turned to 0 degrees
- moved R3 17.8 mm to (104.3, 96.9), turned to 0 degrees
- moved R7 14.4 mm to (88.3, 104.6), turned to 0 degrees
- moved C3 11.9 mm to (92.0, 105.4), turned to -90 degrees
- moved R1 11.6 mm to (104.3, 101.3), turned to 0 degrees
- moved C23 11.5 mm to (94.2, 106.1)
- moved C22 11.5 mm to (94.2, 104.6)
- moved R8 10.4 mm to (97.8, 104.6), turned to 180 degrees
- moved R9 8.60 mm to (90.5, 105.4), turned to -90 degrees
- moved R10 8.56 mm to (92.3, 107.6)
- moved L1 5.39 mm to (87.5, 109.8), turned to 180 degrees
- moved C2 4.87 mm to (89.2, 113.5), turned to 180 degrees
- moved U1 4.75 mm to (92.8, 110.0)
- moved C4 4.55 mm to (84.6, 105.3), turned to 90 degrees
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Connections:
- C2 pad 1: Net-(U1-BST) -> Net-(U1-BOOT)
- C3 pad 1: +3.3V -> Net-(C3-Pad1)
- R1 pad 1: Net-(U4-IPROPI) -> /MOTOR_FAULT
- R1 pad 2: GND -> +3.3V
- R4 pad 1: /MOTOR1 -> /Track_Right
- R4 pad 2: /MOTOR_SENSE_1 -> /DCC
- R5 pad 1: /MOTOR2 -> /DCC
- R5 pad 2: /MOTOR_SENSE_2 -> GND
- R6 pad 1: /MOTOR_SENSE_1 -> Net-(U1-EN)
- R7 pad 1: /MOTOR_SENSE_2 -> +3.3V
- R7 pad 2: GND -> Net-(C3-Pad1)
- R9 pad 1: +3.3V -> Net-(C3-Pad1)
- U1 pad 1: VCC -> GND
- U1 pad 3: GND -> VCC
- U1 pad 4: Net-(U1-BST) -> Net-(U1-FB)
- U1 pad 6: Net-(U1-FB) -> Net-(U1-BOOT)
- U7 pad 31: unconnected-(U7-IO38-Pad31) -> /SCL
- U7 pad 32: unconnected-(U7-MTCK/IO39-Pad32) -> /SDA
- U7 pad 39: /MOTOR_SENSE_1 -> /MOTOR_FAULT
- U7 pad 5: /MOTOR_SENSE_2 -> /DCC
Routing:
- net /MOTOR_FAULT: track 0.00 -> 50.4 mm, vias 0 -> 4
- net /MOTOR2: track 46.8 -> 3.15 mm, vias 1 -> 0
- net /SDA: track 0.00 -> 36.7 mm, vias 0 -> 4
- net /SCL: track 0.00 -> 35.6 mm, vias 0 -> 4
- net /DCC: track 0.00 -> 34.2 mm, vias 0 -> 2
- net /MOTOR1: track 33.0 -> 3.31 mm
- net +3.3V: track 18.8 -> 47.9 mm
- net /MOTOR_SENSE_1: track 25.5 -> 0.00 mm, vias 2 -> 0
- net /BOOT/GPIO C: track 51.7 -> 31.1 mm, vias 3 -> 1
- net /MOTOR_SENSE_2: track 13.9 -> 0.00 mm, vias 2 -> 0
- net /AUX2LED: track 40.9 -> 29.0 mm
- net GND: track 35.4 -> 25.5 mm, vias 24 -> 23
- net /AUX3LED: track 38.1 -> 29.4 mm
- net /AUX4LED: track 36.1 -> 28.0 mm
- net /AUX1LED: track 30.8 -> 23.0 mm
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- added copper zone on F.Cu, net Net-(U1-FB)
Other:
- board size 22.5 x 49.5 mm -> 22.5 x 48.3 mm
- board text added: "AUX2LED | MOTOR1"
- board text added: "AUX3LED | MOTOR2"
- board text added: "AUX4LED | TX/GPIO-A"
- board text added: "BOOT/GPIO-C | RX/GPIO-B"
- board text added: "BackLED | AUX1LED"
- board text added: "FwdLED | +3.3V"
- board text added: "GND | VCC"
- board text added: "MRRDecoder micro v1.0 Pavel Dovgalyuk, 2026"
- board text added: "SMOKE ON"
- board text added: "SOUND1, 2"
- board text added: "TRACK1"
- board text added: "TRACK2"

Commit message: Fixed compiler
Routing:
- net Net-(U1-SW): track 12.3 -> 15.0 mm
- net VCC: vias 3 -> 7
- net GND: vias 23 -> 25
Changed lines of the file:
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@@
 		)
 		(fp_text user "${REFERENCE}"
-			(at 0 0 90)
+			(at 0 0 180)
 			(layer "F.SilkS")
 			(effects
@@
 		)
 		(fp_text user "${REFERENCE}"
-			(at 0 0 90)
-			(layer "F.Fab")
+			(at 0 0 180)
+			(layer "F.SilkS")
 			(effects
 				(font
@@
 		)
 	)
-	(gr_text "SMOKE ON"
-		(at 104.14 102.04 270)
+	(gr_text "TRACK2"
+		(at 104.287457 110.24 270)
 		(layer "B.SilkS")
 		(effects
@@
 		)
 	)
-	(gr_text "TRACK2"
-		(at 104.32 110.03 270)
+	(gr_text "SMOKE ON"
+		(at 104.32 102.1 270)
 		(layer "B.SilkS")
 		(effects
@@
 	)
 	(via
+		(at 90.85 114.86)
+		(size 0.6)
+		(drill 0.3)
+		(layers "F.Cu" "B.Cu")
+		(free yes)
+		(net 1)
+	)
+	(via
 		(at 95.5375 116.92327)
 		(size 0.6)
@@
 	)
 	(via
-		(at 94.84 112.88)
+		(at 94.640166 112.640873)
 		(size 0.6)
 		(drill 0.3)
@@
 	)
 	(via
+		(at 89.17 115.45)
+		(size 0.6)
+		(drill 0.3)
+		(layers "F.Cu" "B.Cu")
+		(free yes)
+		(net 1)
+	)
+	(via
 		(at 92.829514 111.03706)
 		(size 0.4)
@@
 	)
 	(via
-		(at 92.97 114.26)
+		(at 92.37 112.84)
 		(size 0.6)
 		(drill 0.3)
@@
 	)
 	(via
+		(at 95.77 107.94)
+		(size 0.6)
+		(drill 0.3)
+		(layers "F.Cu" "B.Cu")
+		(free yes)
+		(net 2)
+	)
+	(via
 		(at 102.92 109.03)
 		(size 0.6)
@@
 	)
 	(via
+		(at 97.29 107.48)
+		(size 0.6)
+		(drill 0.3)
+		(layers "F.Cu" "B.Cu")
+		(free yes)
+		(net 2)
+	)
+	(via
 		(at 94.04 118.53)
 		(size 0.6)
@@
 	)
 	(via
+		(at 94.52 108.32)
+		(size 0.6)
+		(drill 0.3)
+		(layers "F.Cu" "B.Cu")
+		(free yes)
+		(net 2)
+	)
+	(via
+		(at 99.95 107.46)
+		(size 0.6)
+		(drill 0.3)
+		(layers "F.Cu" "B.Cu")
+		(free yes)
+		(net 2)
+	)
+	(via
 		(at 102.95 111.74)
 		(size 0.6)
@@
 	)
 	(segment
-		(start 88.91 107.86)
-		(end 87.88 108.89)
+		(start 87.85 110.71)
+		(end 87.85 110.803503)
 		(width 1)
 		(layer "In2.Cu")
@@
 	)
 	(segment
-		(start 95.61 108.45)
-		(end 95 107.84)
+		(start 90.876497 113.83)
+		(end 94.544222 113.83)
 		(width 1)
 		(layer "In2.Cu")
@@
 	)
 	(segment
-		(start 95 107.84)
-		(end 94.98 107.86)
+		(start 95.59 110.49)
+		(end 95.59 109.44)
 		(width 1)
 		(layer "In2.Cu")
@@
 	)
 	(segment
-		(start 95.61 109.42)
-		(end 95.61 108.45)
+		(start 87.85 110.71)
+		(end 87.85 108.92)
 		(width 1)
 		(layer "In2.Cu")
@@
 	)
 	(segment
-		(start 94.98 107.86)
-		(end 88.91 107.86)
+		(start 95.79 112.834542)
+		(end 95.79 110.69)
 		(width 1)
 		(layer "In2.Cu")
@@
 	)
 	(segment
-		(start 95.59 110.49)
-		(end 95.59 109.44)
+		(start 87.85 110.803503)
+		(end 90.876497 113.83)
 		(width 1)
 		(layer "In2.Cu")
@@
 	)
 	(segment
-		(start 87.85 110.71)
-		(end 87.85 108.92)
+		(start 95.59 109.44)
+		(end 95.61 109.42)
 		(width 1)
 		(layer "In2.Cu")
@@
 	)
 	(segment
-		(start 95.59 109.44)
-		(end 95.61 109.42)
+		(start 95.79 110.69)
+		(end 95.59 110.49)
+		(width 1)
+		(layer "In2.Cu")
+		(net 5)
+	)
+	(segment
+		(start 94.544222 113.83)
+		(end 94.783349 113.590873)
+		(width 1)
+		(layer "In2.Cu")
+		(net 5)
+	)
+	(segment
+		(start 95.033669 113.590873)
+		(end 95.79 112.834542)
+		(width 1)
+		(layer "In2.Cu")
+		(net 5)
+	)
+	(segment
+		(start 94.783349 113.590873)
+		(end 95.033669 113.590873)
 		(width 1)
 		(layer "In2.Cu")
@@
 		(polygon
 			(pts
-				(xy 94.2 103.86) (xy 92.66 103.86) (xy 92.42 108.58) (xy 92.42 115.22) (xy 104.13 115.27) (xy 104.15 113.21)
-				(xy 102.52 113.21) (xy 102.45 111.28) (xy 103.39 111.29) (xy 103.4 111.32) (xy 103.33 109.47) (xy 95.02 109.47)
-				(xy 95 110.31) (xy 93.18 110.47) (xy 93.16 108.27) (xy 94.24 108.27)
+				(xy 94.2 103.86) (xy 92.66 103.86) (xy 92.42 108.58) (xy 92.42 113.3) (xy 90.73 113.3) (xy 90.72 114.23)
+				(xy 87.76 114.25) (xy 87.77 116.12) (xy 91.31 118.7) (xy 91.26 117.24) (xy 92.42 115.22) (xy 104.13 115.27)
+				(xy 104.15 113.21) (xy 102.52 113.21) (xy 102.45 111.28) (xy 103.39 111.29) (xy 103.4 111.32) (xy 103.33 109.47)
+				(xy 95.02 109.47) (xy 95 110.31) (xy 93.18 110.47) (xy 93.16 108.27) (xy 94.24 108.27)
 			)
 		)
