File: hardware/sounddecoder-esp32-s3-wroom-2-mini/sounddecoder-esp32-s3-wroom-2-mini.kicad_sch (KiCad schematic)
At the start: 34 parts, among them J1 Input power, J10 AUX1, J11 AUX2, J2 Conn_01x02_Pin, J3 Motor, J4 Speaker, J8 FwdLED, J9 BackLED, U1 LM2596S-5, U3 MAX98357A, U4 DRV8251A, U6 AMS1117-3.3, U7 ESP32-S3-WROOM-2, U8 ULN2003A

Commit message: Added gerbers
Parts:
- removed C2: 47uF, Capacitor_SMD:CP_Elec_6.3x5.4, symbol Device:C_Polarized
- added J101: Conn_01x05, Connector_PinHeader_2.54mm:PinHeader_1x05_P2.54mm_Vertical, symbol Connector_Generic:Conn_01x05
Connections:
- net +5V: now also J101.1 (Pin_1)
- net GND: now also J101.5 (Pin_5)
- net IO0: now also J101.4 (Pin_4)
- net MOTOR1: now also J3.1 (Pin_1); no longer J3.2 (Pin_2)
- net MOTOR2: now also J3.2 (Pin_2); no longer J3.1 (Pin_1)
- net UART-RX: now also J101.3 (Pin_3)
- net UART-TX: now also J101.2 (Pin_2)
Other:
- moved on the sheet: C1

Commit message: Added micro board
Parts:
- C1, C10, C11, C12, C3, C7, C8: footprint Capacitor_SMD:C_0805_2012Metric_Pad1.18x1.45mm_HandSolder -> Capacitor_SMD:C_0805_2012Metric
- R1, R2, R3, R4, R5, R6, R7: footprint Resistor_SMD:R_0805_2012Metric_Pad1.20x1.40mm_HandSolder -> Resistor_SMD:R_0805_2012Metric
Changed lines of the file:
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@@
 			)
 		)
-		(property "Footprint" "Resistor_SMD:R_0805_2012Metric_Pad1.20x1.40mm_HandSolder"
+		(property "Footprint" "Resistor_SMD:R_0805_2012Metric"
 			(at 182.118 68.58 90)
 			(effects
@@
 			)
 		)
-		(property "Footprint" "Resistor_SMD:R_0805_2012Metric_Pad1.20x1.40mm_HandSolder"
+		(property "Footprint" "Resistor_SMD:R_0805_2012Metric"
 			(at 75.692 80.01 90)
 			(effects
@@
 			)
 		)
-		(property "Footprint" "Capacitor_SMD:C_0805_2012Metric_Pad1.18x1.45mm_HandSolder"
+		(property "Footprint" "Capacitor_SMD:C_0805_2012Metric"
 			(at 124.1552 109.22 0)
 			(effects
@@
 			)
 		)
-		(property "Footprint" "Capacitor_SMD:C_0805_2012Metric_Pad1.18x1.45mm_HandSolder"
+		(property "Footprint" "Capacitor_SMD:C_0805_2012Metric"
 			(at 27.6352 73.66 0)
 			(effects
@@
 			)
 		)
-		(property "Footprint" "Resistor_SMD:R_0805_2012Metric_Pad1.20x1.40mm_HandSolder"
+		(property "Footprint" "Resistor_SMD:R_0805_2012Metric"
 			(at 130.81 74.168 90)
 			(effects
@@
 			)
 		)
-		(property "Footprint" "Capacitor_SMD:C_0805_2012Metric_Pad1.18x1.45mm_HandSolder"
+		(property "Footprint" "Capacitor_SMD:C_0805_2012Metric"
 			(at 133.6548 76.2 0)
 			(effects
@@
 			)
 		)
-		(property "Footprint" "Capacitor_SMD:C_0805_2012Metric_Pad1.18x1.45mm_HandSolder"
+		(property "Footprint" "Capacitor_SMD:C_0805_2012Metric"
 			(at 135.5852 109.22 0)
 			(effects
@@
 			)
 		)
-		(property "Footprint" "Resistor_SMD:R_0805_2012Metric_Pad1.20x1.40mm_HandSolder"
+		(property "Footprint" "Resistor_SMD:R_0805_2012Metric"
 			(at 87.122 90.17 90)
 			(effects
@@
 			)
 		)
-		(property "Footprint" "Resistor_SMD:R_0805_2012Metric_Pad1.20x1.40mm_HandSolder"
+		(property "Footprint" "Resistor_SMD:R_0805_2012Metric"
 			(at 87.122 76.2 90)
 			(effects
@@
 			)
 		)
-		(property "Footprint" "Resistor_SMD:R_0805_2012Metric_Pad1.20x1.40mm_HandSolder"
+		(property "Footprint" "Resistor_SMD:R_0805_2012Metric"
 			(at 94.742 90.17 90)
 			(effects
@@
 			)
 		)
-		(property "Footprint" "Capacitor_SMD:C_0805_2012Metric_Pad1.18x1.45mm_HandSolder"
+		(property "Footprint" "Capacitor_SMD:C_0805_2012Metric"
 			(at 93.0148 132.08 0)
 			(effects
@@
 			)
 		)
-		(property "Footprint" "Resistor_SMD:R_0805_2012Metric_Pad1.20x1.40mm_HandSolder"
+		(property "Footprint" "Resistor_SMD:R_0805_2012Metric"
 			(at 94.742 76.2 90)
 			(effects
@@
 			)
 		)
-		(property "Footprint" "Capacitor_SMD:C_0805_2012Metric_Pad1.18x1.45mm_HandSolder"
+		(property "Footprint" "Capacitor_SMD:C_0805_2012Metric"
 			(at 30.1752 39.37 0)
 			(effects
@@
 			)
 		)
-		(property "Footprint" "Capacitor_SMD:C_0805_2012Metric_Pad1.18x1.45mm_HandSolder"
+		(property "Footprint" "Capacitor_SMD:C_0805_2012Metric"
 			(at 100.6348 132.08 0)
 			(effects

Commit message: Many updates
Parts:
- removed C4: 470uF, Capacitor_SMD:CP_Elec_10x10.5, symbol Device:C_Polarized
- removed C5: 220uF, Capacitor_SMD:C_Elec_6.3x7.7, symbol Device:C_Polarized
- removed C6: 22uF, Capacitor_SMD:CP_Elec_4x5.4, symbol Device:C_Polarized
- removed D1: SS54, Diode_SMD:D_SMC, symbol Diode:1N5822
- removed J1: Input power, TerminalBlock:TerminalBlock_Xinya_XY308-2.54-2P_1x02_P2.54mm_Horizontal, symbol Connector_Generic:Conn_01x02
- removed J10: AUX1, Connector_PinHeader_2.54mm:PinHeader_1x02_P2.54mm_Vertical, symbol Connector_Generic:Conn_01x02
- removed J101: Conn_01x05, Connector_PinHeader_2.54mm:PinHeader_1x05_P2.54mm_Vertical, symbol Connector_Generic:Conn_01x05
- removed J11: AUX2, Connector_PinHeader_2.54mm:PinHeader_1x02_P2.54mm_Vertical, symbol Connector_Generic:Conn_01x02
- removed J3: Motor, TerminalBlock:TerminalBlock_Xinya_XY308-2.54-2P_1x02_P2.54mm_Horizontal, symbol Connector_Generic:Conn_01x02
- removed J4: Speaker, Connector_PinHeader_2.54mm:PinHeader_1x02_P2.54mm_Vertical, symbol Connector_Generic:Conn_01x02
- removed J8: FwdLED, Connector_PinHeader_2.54mm:PinHeader_1x02_P2.54mm_Vertical, symbol Connector_Generic:Conn_01x02
- removed J9: BackLED, Connector_PinHeader_2.54mm:PinHeader_1x02_P2.54mm_Vertical, symbol Connector_Generic:Conn_01x02
- removed U1: LM2596S-5, Package_TO_SOT_SMD:TO-263-5_TabPin3, symbol Regulator_Switching:LM2596S-5
- removed U4: DRV8251A, Package_SO:Texas_HSOP-8-1EP_3.9x4.9mm_P1.27mm_ThermalVias, symbol Driver_Motor:DRV8231ADSG
- removed U6: AMS1117-3.3, Package_TO_SOT_SMD:SOT-223-3_TabPin2, symbol Regulator_Linear:AMS1117-3.3
- added C12: 47uF, Capacitor_SMD:CP_Elec_6.3x5.4, symbol Device:C_Polarized
- added C14, C2: 0.1uF, Capacitor_SMD:C_0603_1608Metric, symbol Device:C
- added C5: 47pF, Capacitor_SMD:C_0603_1608Metric, symbol Device:C
- added C7, C9: 22uF, Capacitor_SMD:C_0603_1608Metric, symbol Device:C
- added D1, D2, D3, D4: PMEG2020EJ, Diode_SMD:D_SOD-323, symbol PCM_JLCPCB-Diodes:Schottky,B5817WS
- added J1: TrackLeft, TestPoint:TestPoint_THTPad_1.0x1.0mm_Drill0.5mm, symbol Connector:Conn_01x01_Pin
- added J10: Smoke_Pin, TestPoint:TestPoint_THTPad_1.0x1.0mm_Drill0.5mm, symbol Connector:Conn_01x01_Pin
- added J11: Conn_02x11_Odd_Even, Connector_PinHeader_2.00mm:PinHeader_2x11_P2.00mm_Vertical, symbol Connector_Generic:Conn_02x11_Odd_Even
- added J12: Conn_01x06, Connector_PinHeader_2.54mm:PinHeader_1x06_P2.54mm_Vertical, symbol Connector_Generic:Conn_01x06
- added J2: TrackRight, TestPoint:TestPoint_THTPad_1.0x1.0mm_Drill0.5mm, symbol Connector:Conn_01x01_Pin
- added J3, J4, J5, J6, J8, J9: Conn_01x02_Pin, Jumper:SolderJumper-2_P1.3mm_Open_RoundedPad1.0x1.5mm, symbol Connector:Conn_01x02_Pin
- added R10: 100k, Capacitor_SMD:C_0603_1608Metric, symbol Device:R
- added R11: 22.1k, Capacitor_SMD:C_0603_1608Metric, symbol Device:R
- added R14: 511, Capacitor_SMD:C_0603_1608Metric, symbol Device:R
- added R15, R16: 2.2k, Capacitor_SMD:C_0603_1608Metric, symbol Device:R
- added R17: 10k, Capacitor_SMD:C_0603_1608Metric, symbol Device:R
- added R18: 75kΩ, Capacitor_SMD:C_0603_1608Metric, symbol PCM_JLCPCB-Resistors:0402,75kΩ
- added R19: 12kΩ, Capacitor_SMD:C_0603_1608Metric, symbol PCM_JLCPCB-Resistors:0402,20kΩ
- added R2, R3, R8: 30, Capacitor_SMD:C_0603_1608Metric, symbol Device:R
- added R9: 49.9, Capacitor_SMD:C_0603_1608Metric, symbol Device:R
- added U3: TPS54302, Package_TO_SOT_SMD:SOT-23-6, symbol Regulator_Switching:TPS54302
- added U5: DRV8235, Package_DFN_QFN:WQFN-16-1EP_3x3mm_P0.5mm_EP1.68x1.68mm_ThermalVias, symbol custom:DRV8235
- C1: value 0.1uF -> 10uF; footprint Capacitor_SMD:C_0805_2012Metric -> Capacitor_SMD:C_0603_1608Metric
- C10: renamed from C12; footprint Capacitor_SMD:C_0805_2012Metric -> Capacitor_SMD:C_0603_1608Metric
- C11, C3: footprint Capacitor_SMD:C_0805_2012Metric -> Capacitor_SMD:C_0603_1608Metric
- C4: renamed from C8; footprint Capacitor_SMD:C_0805_2012Metric -> Capacitor_SMD:C_0603_1608Metric
- C6: renamed from C7; footprint Capacitor_SMD:C_0805_2012Metric -> Capacitor_SMD:C_0603_1608Metric
- C8: renamed from C10; footprint Capacitor_SMD:C_0805_2012Metric -> Capacitor_SMD:C_0603_1608Metric
- J7: renamed from J2; footprint Connector_PinHeader_1.00mm:PinHeader_1x02_P1.00mm_Vertical -> Jumper:SolderJumper-2_P1.3mm_Open_RoundedPad1.0x1.5mm
- L1: value 47uh/L39 -> 6.8uH; footprint Inductor_SMD:L_Bourns_SRP1245A -> Inductor_SMD:L_Chilisin_BMRA00050530
- R1: value 1k -> 511k; footprint Resistor_SMD:R_0805_2012Metric -> Capacitor_SMD:C_0603_1608Metric
- R12: renamed from R2; footprint Resistor_SMD:R_0805_2012Metric -> Capacitor_SMD:C_0603_1608Metric
- R13: renamed from R3; footprint Resistor_SMD:R_0805_2012Metric -> Capacitor_SMD:C_0603_1608Metric
- R4: value 20k -> 105k; footprint Resistor_SMD:R_0805_2012Metric -> Capacitor_SMD:C_0603_1608Metric
- R5: value 20k -> 30; footprint Resistor_SMD:R_0805_2012Metric -> Capacitor_SMD:C_0603_1608Metric
- R6, R7: value 1k -> 30; footprint Resistor_SMD:R_0805_2012Metric -> Capacitor_SMD:C_0603_1608Metric
- renumbered U8 to U1, U3 to U2, U7 to U4
Connections:
- net +5V is gone; now on net +3.3V: L1.2, U1.9 (COM)
- net +3.3V: now also C14.1, C7.1, C9.1, J11.18 (Pin_18), J11.20 (Pin_20), J11.22 (Pin_22), J11.4 (Pin_4), R15.1, R16.1, R17.2, R9.1, U5.11 (~{SLEEP}), U5.16 (VREF)
- net GND: now also R4.2, C12.2, C14.2, C2.2, C7.2, C9.2, D3.2, D4.2, J11.15 (Pin_15), J12.6 (Pin_6), R11.2, R14.2, R19.2, U3.1 (GND), U5.10 (A0), U5.17 (GND(PPAD)), U5.7 (GND), U5.9 (A1); no longer C3.2, R1.2, R6.2, R7.2
- net MOTOR1: now also J11.8 (Pin_8), J12.3 (Pin_3), U5.6 (OUT1); no longer R4.1
- net MOTOR2: now also J11.10 (Pin_10), J12.4 (Pin_4), U5.8 (OUT2); no longer R5.1
- net VCC: now also R1.1, C12.1, C2.1, D1.1, D2.1, J11.16 (Pin_16), J12.5 (Pin_5), U3.3 (VIN), U5.5 (VM); no longer C3.1
- net OUT1: now reaches U1.1 (I1)
- net OUT1: now also U4.25 (IO48)
- net at U1.10 (O7): now also J8.1 (Pin_1), R8.1
- net at U1.11 (O6): now also J3.1 (Pin_1), R3.1
- net at U1.12 (O5): now also R6.1, J5.1 (Pin_1)
- net at U1.13 (O4): now also R7.1, J9.2 (Pin_2)
- net SmokeOn: now reaches U1.16 (O1)
- net SmokeOn: now also J10.1 (Pin_1)
- net OUT6: now reaches U1.6 (I6)
- net OUT6: now also U4.20 (IO12)
- net OUT7: now reaches U1.7 (I7)
- net OUT7: now also U4.19 (IO11)
- net GPIO J: now reaches U4.10 (IO17)
- net GPIO K: now reaches U4.11 (IO18)
- net GPIO G: now reaches U4.12 (IO8)
- net GPIO F: now reaches U4.18 (IO10)
- net GPIO F: now also J11.7 (Pin_7)
- net SCL: now reaches U4.31 (IO38)
- net SCL: now also R15.2, U5.15 (SCL)
- net SDA: now reaches U4.32 (MTCK/IO39)
- net SDA: now also R16.2, U5.14 (SDA)
- net GPIO E: now reaches U4.6 (IO6)
- net GPIO E: now also J11.5 (Pin_5)
- net GPIO D: now reaches U4.7 (IO7)
- net GPIO D: now also J11.3 (Pin_3)
- net GPIO H: now reaches U4.8 (IO15)
- net GPIO I: now reaches U4.9 (IO16)
- net BackLED: no longer names the net of U1.14 (O3)
- net BackLED: now also R5.1, J6.2 (Pin_2)
- net FwdLED: no longer names the net of U1.15 (O2)
- net FwdLED: now also J4.2 (Pin_2), R2.1
- net IO0 renamed BOOT/GPIO C
- net BOOT/GPIO C: now also J11.6 (Pin_6)
- net MOTOR_IN1: no longer names the net of U4.38 (IO2)
- net MOTOR_IN2: no longer names the net of U4.4 (IO4)
- removed net MOTOR_SENSE_1: R4.2, R6.1, U4.39 (IO1)
- removed net MOTOR_SENSE_2: R5.2, R7.1, U4.5 (IO5)
- net Out5V: no longer names the net of L1.1
- net Out5V: now also C3.2, U3.2 (SW)
- net Sound1 renamed SOUND1
- net SOUND1: now also J11.1 (Pin_1), J12.1 (Pin_1)
- net Sound2 renamed SOUND2
- net SOUND2: now also J11.2 (Pin_2), J12.2 (Pin_2)
- net UART-RX renamed UART-RX/GPIO B
- net UART-RX/GPIO B: now also J11.14 (Pin_14)
- net UART-TX renamed UART-TX/GPIO A
- net UART-TX/GPIO A: now also J11.12 (Pin_12)
- new net: R1.2, R4.1, U3.5 (EN)
- new net: C5.1, R10.1, R9.2
- new net: C5.2, R10.2, R11.1, U3.4 (FB)
- new net: C3.1, U3.6 (BOOT)
- new net: R14.1, U5.1 (IPROPI)
- new net DCC: R18.2, R19.1, U4.5 (IO5)
- new net LED1: J11.21 (Pin_21), J4.1 (Pin_1), R2.2
- new net LED2: J11.19 (Pin_19), J6.1 (Pin_1), R5.2
- new net LED3: J11.17 (Pin_17), J9.1 (Pin_1), R7.2
- new net LED4: J11.13 (Pin_13), J5.2 (Pin_2), R6.2
- new net LED5: J11.11 (Pin_11), J3.2 (Pin_2), R3.2
- new net LED6: J11.9 (Pin_9), J8.2 (Pin_2), R8.2
- new net MOTOR_FAULT: R17.1, U4.39 (IO1), U5.4 (~{FAULT})
- new net Track_Left: D1.2, D4.1, J1.1 (Pin_1)
- new net Track_Right: D2.2, D3.1, J2.1 (Pin_1), R18.1
- no-connect marks 0 -> 10
Other:
- note added: "Many other capacitors on power."
- moved on the sheet: C4, C6, J7, U2
